Commit message: adding simulation controllers for the jetbot

File: simulation_ws/src/jetbot_urdf_with_controllers_and_launch/jetbot_description/urdf/jetbot.urdf (robot description, URDF)
Before this commit: robot JetBot, 4 links, 3 joints
Links:
- link JetBot__chassis: mass 0 -> 0.5
- link JetBot__left_wheel: mass 0 -> 0.01
- link JetBot__right_wheel: mass 0 -> 0.01
Joints:
- joint JetBot__left_wheel_hinge: type fixed -> continuous
- joint JetBot__right_wheel_hinge: type fixed -> continuous

Commit message: adds default limits for the model

File: simulation_ws/src/jetbot_urdf_with_controllers_and_launch/jetbot_description/urdf/jetbot.urdf (robot description, URDF)
Before this commit: robot JetBot, 4 links, 3 joints
Joints:
- joint JetBot__left_wheel_hinge: limit lower=0 upper=0 effort=0 velocity=0 -> effort=30 velocity=1.0
- joint JetBot__right_wheel_hinge: limit lower=0 upper=0 effort=0 velocity=0 -> effort=30 velocity=1.0

Commit message: updates inertial values and mass

File: simulation_ws/src/jetbot_urdf_with_controllers_and_launch/jetbot_description/urdf/jetbot.urdf (robot description, URDF)
Before this commit: robot JetBot, 4 links, 3 joints
Links:
- link JetBot__chassis: mass 0.5 -> 5.0
- link JetBot__left_wheel: mass 0.01 -> 1.5
- link JetBot__right_wheel: mass 0.01 -> 1.5
Joints:
- joint JetBot__camera_joint: limit lower=0 upper=0 effort=0 velocity=0 -> (none)

Commit message: minor changes to mass

File: simulation_ws/src/jetbot_urdf_with_controllers_and_launch/jetbot_description/urdf/jetbot.urdf (robot description, URDF)
Before this commit: robot JetBot, 4 links, 3 joints
Links:
- link JetBot__chassis: mass 5.0 -> 2.5
- link JetBot__left_wheel: mass 1.5 -> 0.5
- link JetBot__right_wheel: mass 1.5 -> 0.5

Commit message: updates the jetbot control with a DiffDriveController to enable better motion

File: simulation_ws/src/jetbot_urdf_with_controllers_and_launch/jetbot_description/urdf/jetbot.urdf (robot description, URDF)
Before this commit: robot JetBot, 4 links, 3 joints
Links:
- link JetBot__chassis: mass 2.5 -> 1.0
- link JetBot__left_wheel: geometry collision cylinder length=0.008 radius=0.030; visual mesh filename=package://jetbot_description/meshes/JetBot-v3-Wheel.stl scale=0.001 0.001 0.001
- link JetBot__right_wheel: geometry collision cylinder length=0.008 radius=0.030; visual mesh filename=package://jetbot_description/meshes/JetBot-v3-Wheel.stl scale=0.001 0.001 0.001

Commit message: cleanup

File: simulation_ws/src/jetbot_urdf_with_controllers_and_launch/jetbot_description/urdf/jetbot.urdf (robot description, URDF)
Before this commit: robot JetBot, 4 links, 3 joints
Links:
- link JetBot__camera_link: mass 0.1 -> 0.01
- link JetBot__left_wheel: mass 0.5 -> 0.1
- link JetBot__right_wheel: mass 0.5 -> 0.1
Joints:
- joint JetBot__left_wheel_hinge: limit effort=30 velocity=1.0 -> (none)
- joint JetBot__right_wheel_hinge: limit effort=30 velocity=1.0 -> (none)
